Commit message: gazebo仿真二（添加了laser插件）

File: src/rm_description/urdf/rm_sentry/actuator/caster.urdf.xacro (robot description, xacro)
@@ -3,40 +3,47 @@
     <xacro:include filename="$(find rm_description)/urdf/rm_sentry/common_inertia.xacro" />
     <!-- 机器人的IMU部件，惯性测量传感器 -->
-    <xacro:macro name="imu_xacro" params="xyz">
-        <link name="imu_link">
+    <xacro:macro name="caster_xacro" params="caster_name xyz">
+        <link name="${caster_name}_link">
             <!-- 部件外观 -->
             <visual>
                 <!-- 沿着自己几何中心的偏移（xyz）和旋转（roll,pitch,yaw） ，用origin来定义-->
-                <origin xyz="0.0 0.0 0.0" rpy="0.0 0.0 0.0"/>
+                <origin xyz="0.0 0.0 0.0" rpy="1.57079 0.0 0.0"/>
                 <!-- 几何形状 ，用geometry来定义-->
                 <geometry>
                     <!-- cylinder（圆柱体），radius(半径)，length(高度) -->
-                    <box size="0.02 0.02 0.02"/>
+                    <sphere radius="0.016"/>
                 </geometry>
                 <!-- 材质颜色描述 ，用material定义-->
-                <material name="white">
-                    <color rgba="0.0 0.0 0.0 0.5"/>
+                <material name="yellow">
+                    <color rgba="1.0 1.0 0.0 0.8"/>
                 </material>
             </visual>
             <collision>
                 <!-- 沿着自己几何中心的偏移（xyz）和旋转（roll,pitch,yaw） ，用origin来定义-->
-                <origin xyz="0.0 0.0 0.0" rpy="0.0 0.0 0.0"/>
+                <origin xyz="0.0 0.0 0.0" rpy="1.57079 0.0 0.0"/>
                 <!-- 几何形状 ，用geometry来定义-->
                 <geometry>
                     <!-- cylinder（圆柱体），radius(半径)，length(高度) -->
-                    <box size="0.02 0.02 0.02"/>
+                    <sphere radius="0.016"/>
                 </geometry>
                 <!-- 材质颜色描述 ，用material定义-->
-                <material name="white">
-                    <color rgba="0.0 0.0 0.0 0.5"/>
+                <material name="yellow">
+                    <color rgba="1.0 1.0 0.0 0.8"/>
                 </material>
             </collision>
-            <xacro:box_inertia m = "0.02" w = "0.02" h = "0.02" d = "0.02"/>
+            <xacro:sphere_inertia m = "0.05" r = "0.016" />
         </link>
-        <joint name="imu_joint" type="fixed">
-            <origin xyz="${xyz}" rpy="0.0 0.0 0.0"/>
+        <joint name="${caster_name}_joint" type="fixed">
+            <origin xyz="${xyz}" rpy = "0.0 0.0 0.0"/>
             <parent link="base_link"/>
-            <child link="imu_link"/>
+            <child link="${caster_name}_link"/>
         </joint>
+        <gazebo reference = "${caster_name}_link">
+            <mu1 value="0.0"/>
+            <mu2 value="0.0"/>
+            <kp value="1000000000.0"/>
+            <kd value="1.0"/>
+            <material>Gazebo/Black</material>
+        </gazebo>
     </xacro:macro>
 </robot>

File: src/rm_description/urdf/rm_sentry/actuator/whell.urdf.xacro (robot description, xacro)
@@ -3,40 +3,48 @@
     <xacro:include filename="$(find rm_description)/urdf/rm_sentry/common_inertia.xacro" />
     <!-- 机器人的IMU部件，惯性测量传感器 -->
-    <xacro:macro name="imu_xacro" params="xyz">
-        <link name="imu_link">
+    <xacro:macro name="whell_xacro" params="whell_name xyz">
+        <link name="${whell_name}_link">
             <!-- 部件外观 -->
             <visual>
                 <!-- 沿着自己几何中心的偏移（xyz）和旋转（roll,pitch,yaw） ，用origin来定义-->
-                <origin xyz="0.0 0.0 0.0" rpy="0.0 0.0 0.0"/>
+                <origin xyz="0.0 0.0 0.0" rpy="1.57079 0.0 0.0"/>
                 <!-- 几何形状 ，用geometry来定义-->
                 <geometry>
                     <!-- cylinder（圆柱体），radius(半径)，length(高度) -->
-                    <box size="0.02 0.02 0.02"/>
+                    <cylinder radius="0.032" length="0.04"/>
                 </geometry>
                 <!-- 材质颜色描述 ，用material定义-->
-                <material name="white">
-                    <color rgba="0.0 0.0 0.0 0.5"/>
+                <material name="yellow">
+                    <color rgba="1.0 1.0 0.0 0.8"/>
                 </material>
             </visual>
             <collision>
                 <!-- 沿着自己几何中心的偏移（xyz）和旋转（roll,pitch,yaw） ，用origin来定义-->
-                <origin xyz="0.0 0.0 0.0" rpy="0.0 0.0 0.0"/>
+                <origin xyz="0.0 0.0 0.0" rpy="1.57079 0.0 0.0"/>
                 <!-- 几何形状 ，用geometry来定义-->
                 <geometry>
                     <!-- cylinder（圆柱体），radius(半径)，length(高度) -->
-                    <box size="0.02 0.02 0.02"/>
+                    <cylinder radius="0.032" length="0.04"/>
                 </geometry>
                 <!-- 材质颜色描述 ，用material定义-->
-                <material name="white">
-                    <color rgba="0.0 0.0 0.0 0.5"/>
+                <material name="yellow">
+                    <color rgba="1.0 1.0 0.0 0.8"/>
                 </material>
             </collision>
-            <xacro:box_inertia m = "0.02" w = "0.02" h = "0.02" d = "0.02"/>
+            <xacro:cylinder_inertia m = "0.05" r = "0.032" h = "0.04" />
         </link>
-        <joint name="imu_joint" type="fixed">
-            <origin xyz="${xyz}" rpy="0.0 0.0 0.0"/>
+        <joint name="${whell_name}_joint" type="continuous">
+            <origin xyz="${xyz}" rpy = "0.0 0.0 0.0"/>
             <parent link="base_link"/>
-            <child link="imu_link"/>
+            <child link="${whell_name}_link"/>
+            <axis xyz="0 1 0"/>
         </joint>
+        <gazebo reference = "${whell_name}_link">
+            <mu1 value="20.0"/>
+            <mu2 value="20.0"/>
+            <kp value="1000000000.0"/>
+            <kd value="1.0"/>
+            <material>Gazebo/Black</material>
+        </gazebo>
     </xacro:macro>
 </robot>

File: src/rm_description/urdf/rm_sentry/base.urdf.xacro (robot description, xacro)
@@ -1,5 +1,8 @@
 <?xml version="1.0"?>
 <robot xmlns:xacro="http://www.ros.org/wiki/xacro" >
+    <xacro:include filename="$(find rm_description)/urdf/rm_sentry/common_inertia.xacro" />
     <xacro:macro name="base_xacro" params="radius length">
+        <link name = "base_footprint">
+        </link>
         <link name="base_link">
             <!-- 部件外观 -->
@@ -17,5 +20,24 @@
                 </material>
             </visual>
+            <collision>
+                <!-- 沿着自己几何中心的偏移（xyz）和旋转（roll,pitch,yaw） ，用origin来定义-->
+                <origin xyz="0.0 0.0 0.0" rpy="0.0 0.0 0.0"/>
+                <!-- 几何形状 ，用geometry来定义-->
+                <geometry>
+                    <!-- cylinder（圆柱体），radius(半径)，length(高度) -->
+                    <cylinder radius="${radius}" length="${length}"/>
+                </geometry>
+                <!-- 材质颜色描述 ，用material定义-->
+                <material name="white">
+                    <color rgba="1.0 1.0 1.0 0.5"/>
+                </material>
+            </collision>
+            <xacro:cylinder_inertia m = "1.0" r = "${radius}" h = "${length}" />
         </link>
+        <joint name="base_footprint_joint" type="fixed">
+            <origin xyz="0.0 0.0 ${length/2.0 + 0.032 - 0.001}" rpy="0.0 0.0 0.0"/>
+            <parent link="base_footprint"/>
+            <child link="base_link"/>
+        </joint>
     </xacro:macro>
 </robot>

File: src/rm_description/urdf/rm_sentry/rm_sentry.urdf.xacro (robot description, xacro)
@@ -5,7 +5,20 @@
 <xacro:include filename="$(find rm_description)/urdf/rm_sentry/sensor/camera.urdf.xacro" />
 <xacro:include filename="$(find rm_description)/urdf/rm_sentry/sensor/laser.urdf.xacro" />
+<xacro:include filename="$(find rm_description)/urdf/rm_sentry/sensor/laser.urdf.xacro" />
+<xacro:include filename="$(find rm_description)/urdf/rm_sentry/actuator/whell.urdf.xacro" />
+<xacro:include filename="$(find rm_description)/urdf/rm_sentry/actuator/caster.urdf.xacro" />
+<xacro:include filename="$(find rm_description)/urdf/rm_sentry/plugins/gazebo_control_plugin.xacro" />
+<xacro:include filename="$(find rm_description)/urdf/rm_sentry/plugins/gazebo_sensor_plugin.xacro" />
+<!-- 传感器部分 -->
 <xacro:base_xacro radius = "0.25" length = "0.45" />
 <xacro:imu_xacro xyz = "0.0 0.0 0.15" />
 <xacro:laser_xacro xyz = "0.0 0.0 0.35" />
 <!-- <xacro:camera_xacro xyz = "0.125 0.0 0.0" /> -->
+<!-- 执行器部分 -->
+<xacro:whell_xacro whell_name = "left_whell" xyz = "0.0 0.25 -0.225" />
+<xacro:whell_xacro whell_name = "right_whell" xyz = "0.0 -0.25 -0.225" />
+<xacro:caster_xacro caster_name = "front_caster" xyz = "0.21 0.0 -0.241" />
+<xacro:caster_xacro caster_name = "back_caster" xyz = "-0.21 0.0 -0.241" />
+<xacro:gazebo_control_plugin />
+<xacro:gazebo_sensor_plugin />
 </robot>

File: src/rm_description/urdf/rm_sentry/sensor/laser.urdf.xacro (robot description, xacro)
@@ -1,4 +1,5 @@
 <?xml version="1.0"?>
 <robot xmlns:xacro="http://www.ros.org/wiki/xacro" >
+    <xacro:include filename="$(find rm_description)/urdf/rm_sentry/common_inertia.xacro" />
     <!-- 雷达 -->
     <xacro:macro name="laser_xacro" params="xyz">
@@ -18,4 +19,18 @@
                 </material>
             </visual>
+            <collision>
+                <!-- 沿着自己几何中心的偏移（xyz）和旋转（roll,pitch,yaw） ，用origin来定义-->
+                <origin xyz="0.0 0.0 0.0" rpy="0.0 0.0 0.0"/>
+                <!-- 几何形状 ，用geometry来定义-->
+                <geometry>
+                    <!-- cylinder（圆柱体），radius(半径)，length(高度) -->
+                    <cylinder radius="0.03" length="0.06"/>
+                </geometry>
+                <!-- 材质颜色描述 ，用material定义-->
+                <material name="black">
+                    <color rgba="0.0 0.0 0.0 1.0"/>
+                </material>
+            </collision>
+            <xacro:cylinder_inertia m = "0.10" r = "0.03" h = "0.06" />
         </link>
         <!-- 雷达支撑杆 -->
@@ -30,4 +45,14 @@
                 </material>
             </visual>
+            <collision>
+                <origin xyz="0.0 0.0 0.0" rpy="0.0 0.0 0.0"/>
+                <geometry>
+                    <cylinder radius="0.01" length="0.25"/>
+                </geometry>
+                <material name="black">
+                    <color rgba="0.0 0.0 0.0 1.0"/>
+                </material>
+            </collision>
+            <xacro:cylinder_inertia m = "0.05" r = "0.01" h = "0.25" />
         </link>
         <!-- 雷达支撑 joint -->
@@ -44,4 +69,10 @@
             <child link="laser_link"/>
         </joint>
+        <gazebo reference = "laser_cylinder_link">
+            <material>Gazebo/Black</material>
+        </gazebo>
+        <gazebo reference = "laser_link">
+            <material>Gazebo/Black</material>
+        </gazebo>
     </xacro:macro>
 </robot>
