Commit message: 1

File: src/rm_description/urdf/fishbot/fishbot.urdf.xacro (robot description, xacro)
@@ -2,18 +2,23 @@
 <robot xmlns:xacro="http://www.ros.org/wiki/xacro" name="fishbot">
     <xacro:include filename="$(find rm_description)/urdf/fishbot/base.urdf.xacro" />
+    <!-- 传感器组件 -->
     <xacro:include filename="$(find rm_description)/urdf/fishbot/sensor/imu.urdf.xacro" />
     <xacro:include filename="$(find rm_description)/urdf/fishbot/sensor/laser.urdf.xacro" />
     <xacro:include filename="$(find rm_description)/urdf/fishbot/sensor/camera.urdf.xacro" />
+     <!-- 执行器组件 -->
     <xacro:include filename="$(find rm_description)/urdf/fishbot/actuator/wheel.urdf.xacro" />
     <xacro:include filename="$(find rm_description)/urdf/fishbot/actuator/caster.urdf.xacro" />
-    <xacro:base_xacro length="0.12" radius="0.25" />
+    <xacro:base_xacro length="0.12" radius="0.1" />
+    <!-- 传感器 -->
     <xacro:imu_xacro xyz="0 0 0.02" />
-    <xacro:laser_xacro xyz="0 0 0.25" />
+    <xacro:laser_xacro xyz="0 0 0.10" />
     <xacro:camera_xacro xyz="0.10 0 0.075" />
+    <!-- 执行器主动轮+从动轮 -->
     <xacro:wheel_xacro wheel_name="left" xyz="0 0.10 -0.06" />
     <xacro:wheel_xacro wheel_name="right" xyz="0 -0.10 -0.06" />
     <xacro:caster_xacro caster_name="front" xyz="0.08 0.0 -0.076" />
     <xacro:caster_xacro caster_name="back" xyz="-0.08 0.0 -0.076" />
-    <!-- <xacro:include filename="$(find rm_description)/urdf/fishbot/plugins/gazebo_control_plugin.xacro" /> -->
+    <!-- Gazebo 插件 -->
+    <xacro:include filename="$(find rm_description)/urdf/fishbot/plugins/gazebo_control_plugin.xacro" />
     <!-- <xacro:gazebo_control_plugin /> -->
     <xacro:include filename="$(find rm_description)/urdf/fishbot/fishbot.ros2_control.xacro" />

File: src/rm_description/urdf/fishbot/plugins/gazebo_sensor_plugin.xacro (robot description, xacro)
@@ -4,31 +4,34 @@
         <gazebo reference="laser_link">
             <sensor name="laserscan" type="ray">
+                <plugin name="laserscan" filename="libgazebo_ros_ray_sensor.so">
+                    <ros>
+                        <namespace>/</namespace>
+                        <remapping>~/out:=scan</remapping>
+                    </ros>
+                    <output_type>sensor_msgs/LaserScan</output_type>
+                    <frame_name>laser_link</frame_name>
+                </plugin>
                 <always_on>true</always_on>
-                <!-- <visualize>true</visualize> -->
                 <visualize>true</visualize>
-                <update_rate>10</update_rate>
+                <update_rate>5</update_rate>
                 <pose>0 0 0 0 0 0</pose>
+								<!-- 激光传感器配置 -->
                 <ray>
+                    <!-- 设置扫描范围 -->
                     <scan>
-                    <!-- Horizontal scan (360 deg) -->
-                    <horizontal>
-                        <samples>720</samples>
-                        <resolution>1</resolution>
-                        <min_angle>-3.1415926</min_angle>
-                        <max_angle>3.1415926</max_angle>
-                    </horizontal>
-                    <!-- Vertical scan (3D) -->
-                    <vertical>
-                        <samples>16</samples>
-                        <resolution>1</resolution>
-                        <min_angle>-0.907571</min_angle>
-                        <max_angle>0.122173</max_angle>
-                    </vertical>
+                        <horizontal>
+                            <samples>360</samples>
+                            <resolution>1.000000</resolution>
+                            <min_angle>0.000000</min_angle>
+                            <max_angle>6.280000</max_angle>
+                        </horizontal>
                     </scan>
+                    <!-- 设置扫描距离 -->
                     <range>
-                        <min>0.12</min>
-                        <max>25.0</max>
-                        <resolution>0.02</resolution>
+                        <min>0.120000</min>
+                        <max>8.0</max>
+                        <resolution>0.015000</resolution>
                     </range>
+                    <!-- 设置噪声 -->
                     <noise>
                         <type>gaussian</type>
@@ -37,14 +40,4 @@
                     </noise>
                 </ray>
-                <!-- ROS2 bridge -->
-                <plugin name="laserscan_ros"
-                        filename="libgazebo_ros_ray_sensor.so">
-                    <ros>
-                        <namespace>/</namespace>
-                        <remapping>~/out:=livox/lidar</remapping>
-                    </ros>
-                    <output_type>sensor_msgs/PointCloud2</output_type>
-                    <frame_name>laser_link</frame_name>
-                </plugin>
             </sensor>
         </gazebo>

File: src/rm_description/urdf/fishbot/sensor/laser.urdf.xacro (robot description, xacro)
@@ -9,9 +9,10 @@
             <material>Gazebo/Black</material>
         </gazebo>
+        <!-- ============雷达支撑杆================ -->
         <link name="laser_cylinder_link">
             <visual>
                 <origin xyz="0 0 0" rpy="0 0 0" />
                 <geometry>
-                    <cylinder length="0.40" radius="0.01" />
+                    <cylinder length="0.10" radius="0.01" />
                 </geometry>
                 <material name="black">
@@ -22,5 +23,5 @@
                 <origin xyz="0 0 0" rpy="0 0 0" />
                 <geometry>
-                    <cylinder length="0.40" radius="0.01" />
+                    <cylinder length="0.10" radius="0.01" />
                 </geometry>
                 <material name="black">
@@ -35,4 +36,5 @@
             <origin xyz="${xyz}" />
         </joint>
+        <!-- ============雷达================ -->
         <link name="laser_link">
             <visual>
@@ -59,5 +61,5 @@
             <parent link="laser_cylinder_link" />
             <child link="laser_link" />
-            <origin xyz="0 0 0.20" />
+            <origin xyz="0 0 0.05" />
         </joint>
     </xacro:macro>

Commit message: 2D雷达

File: src/rm_description/urdf/fishbot/fishbot.urdf.xacro (robot description, xacro)
@@ -12,5 +12,5 @@
     <!-- 传感器 -->
     <xacro:imu_xacro xyz="0 0 0.02" />
-    <xacro:laser_xacro xyz="0 0 0.10" />
+    <xacro:laser_xacro xyz="0 0 0.08" />
     <xacro:camera_xacro xyz="0.10 0 0.075" />
     <!-- 执行器主动轮+从动轮 -->

File: src/rm_description/urdf/fishbot/sensor/laser.urdf.xacro (robot description, xacro)
@@ -14,5 +14,5 @@
                 <origin xyz="0 0 0" rpy="0 0 0" />
                 <geometry>
-                    <cylinder length="0.10" radius="0.01" />
+                    <cylinder length="0.05" radius="0.01" />
                 </geometry>
                 <material name="black">
@@ -23,5 +23,5 @@
                 <origin xyz="0 0 0" rpy="0 0 0" />
                 <geometry>
-                    <cylinder length="0.10" radius="0.01" />
+                    <cylinder length="0.05" radius="0.01" />
                 </geometry>
                 <material name="black">
@@ -61,5 +61,5 @@
             <parent link="laser_cylinder_link" />
             <child link="laser_link" />
-            <origin xyz="0 0 0.05" />
+            <origin xyz="0 0 0.025" />
         </joint>
     </xacro:macro>
