Commit message: 创建了以雷达为基坐标系的tf树

File: src/rm_description/urdf/sentry.urdf (robot description, URDF)
Before this commit: robot sentry, 7 links, 6 joints
Joints:
- joint base_footprint_joint: child classis -> base_footprint; origin xyz=0 0 0.05 rpy=0 0 0 -> xyz=0 0 -0.05 rpy=0 0 0; parent base_footprint -> classis
- joint gimbal_yaw: child gimbal -> classis; origin xyz=0 0 0.131815 rpy=0 0 0 -> xyz=0 0 -0.131815 rpy=0 0 0; parent classis -> gimbal
- joint livox_frame_frame: child livox_frame -> gimbal; origin xyz=0 0.150917 0.17494 rpy=-1.5708 0 0 -> xyz=0 0.17494 -0.150917 rpy=1.5708 0 0; parent gimbal -> livox_frame

Commit message: 增加stalker

File: src/rm_description/urdf/sentry.urdf (robot description, URDF)
Before this commit: robot sentry, 7 links, 6 joints
Joints:
- removed joint camera
- removed joint gimbal_pitch
- removed joint imu_up_frame
- removed joint livox_frame_frame
- added joint camera_joint: type fixed, parent classis, child camera, origin xyz=0.0326601 0 0.3767652 rpy=0 0.00152726 0, axis 0 0 0
- added joint imu_up_joint: type fixed, parent classis, child imu_up, origin xyz=0.0326601 0 0.3242652 rpy=0 0.00152726 0, axis 0 0 0
- added joint livox_frame_joint: type fixed, parent livox_frame, child base_footprint, origin xyz=0 0.356755 -0.150917 rpy=1.5708 0 0, axis 0 0 0
- added joint muzzle_joint: type fixed, parent classis, child muzzle, origin xyz=0 -0.105 0.306815 rpy=0 0.00152726 0, axis 0 0 0
- joint base_footprint_joint: child base_footprint -> classis; origin xyz=0 0 -0.05 rpy=0 0 0 -> xyz=0 0 0.05 rpy=0 0 0; parent classis -> base_footprint
- joint gimbal_yaw: child classis -> gimbal; origin xyz=0 0 -0.131815 rpy=0 0 0 -> xyz=0 0 0.131815 rpy=0 0 0; parent gimbal -> classis
